Commit message: fix: Scale torso STLs by 0.001 and correct all joint origins/rotations

File: src/dual_arm_torso/urdf/dual_arm_torso.urdf.xacro (robot description, xacro)
@@ -6,5 +6,5 @@
       <visual>
         <geometry>
-          <mesh filename="package://dual_arm_torso/meshes/assembly_main_simplified.STL"/>
+          <mesh filename="package://dual_arm_torso/meshes/assembly_main_simplified.STL" scale="0.001 0.001 0.001"/>
         </geometry>
         <material name="torso_gray">
@@ -35,5 +35,5 @@
       <visual>
         <geometry>
-          <mesh filename="package://dual_arm_torso/meshes/mts_carriage.STL"/>
+          <mesh filename="package://dual_arm_torso/meshes/mts_carriage.STL" scale="0.001 0.001 0.001"/>
         </geometry>
         <material name="carriage_dark">
@@ -59,5 +59,5 @@
       <!-- The STL X range is -309 to +257. Let's put left carriage at X=-200, Y=100 -->
       <!-- We might need to rotate it if it faces the wrong way. -->
-      <origin xyz="-0.200 0.100 0.050" rpy="0 0 0"/>
+      <origin xyz="-0.150 0.284 0.050" rpy="0 0 0"/>
       <axis xyz="0 0 1"/>
       <limit lower="0.05" upper="0.8" effort="100.0" velocity="0.5"/>
@@ -67,5 +67,5 @@
       <visual>
         <geometry>
-          <mesh filename="package://dual_arm_torso/meshes/mts_carriage.STL"/>
+          <mesh filename="package://dual_arm_torso/meshes/mts_carriage.STL" scale="0.001 0.001 0.001"/>
         </geometry>
         <material name="carriage_dark">
@@ -89,5 +89,5 @@
       <child link="right_carriage_link"/>
       <!-- Estimated position of the right rail. -->
-      <origin xyz="0.150 0.100 0.050" rpy="0 0 0"/>
+      <origin xyz="0.150 0.284 0.050" rpy="0 0 0"/>
       <axis xyz="0 0 1"/>
       <limit lower="0.05" upper="0.8" effort="100.0" velocity="0.5"/>

File: src/pas_dual_arm_bringup/urdf/robot.urdf.xacro (robot description, xacro)
@@ -6,5 +6,5 @@
   <!-- 1. OMNI BASE -->
   <!-- We include the omni_base description. It provides the base_link and wheels. -->
-  <xacro:include filename="$(find omni_base_description)/urdf/omni_base.urdf.xacro"/>
+  <xacro:include filename="$(find omni_base_description)/robots/omni_base.urdf.xacro"/>
   <!-- 2. DUAL ARM TORSO -->
   <!-- We include our custom torso and attach it to the base_link -->
@@ -13,5 +13,5 @@
        Let's place it at the center of the base, somewhat elevated. -->
   <xacro:dual_arm_torso parent="base_footprint">
-    <origin xyz="0 0 0.2" rpy="0 0 0"/>
+    <origin xyz="0 0 0.2" rpy="0 0 -1.5708"/>
   </xacro:dual_arm_torso>
   <!-- 3. KINOVA GEN3 ARMS -->
@@ -34,5 +34,5 @@
     connection_inactivity_timeout_ms="2000"
     sim_ignition="$(arg sim_ignition)">
-    <origin xyz="0.06 0.02 0.11" rpy="0 1.5708 0"/>
+    <origin xyz="0.060 0.047 0.112" rpy="-1.5708 0 0"/>
   </xacro:load_robot>
   <!-- Right Arm -->
@@ -53,5 +53,5 @@
     connection_inactivity_timeout_ms="2000"
     sim_ignition="$(arg sim_ignition)">
-    <origin xyz="0.06 0.02 0.11" rpy="0 1.5708 0"/>
+    <origin xyz="0.060 0.047 0.112" rpy="-1.5708 0 0"/>
   </xacro:load_robot>
   <!-- 4. PAN-TILT & REALSENSE -->
@@ -60,5 +60,5 @@
   <xacro:pan_tilt parent="torso_base_link">
     <!-- Place the pan-tilt at the top of the torso (Z=0.956) -->
-    <origin xyz="0 0 0.956" rpy="0 0 0"/>
+    <origin xyz="0 0 0.956" rpy="0 0 1.5708"/>
   </xacro:pan_tilt>
   <!-- Include Realsense D435 camera URDF -->
@@ -66,5 +66,5 @@
   <xacro:include filename="$(find realsense2_description)/urdf/_d435.urdf.xacro"/>
   <!-- Attach the camera to the pan_tilt top link -->
-  <xacro:sensor_d435 parent="tilt_link" name="camera" use_nominal_extrinsics="true">
+  <xacro:sensor_d435 parent="pan_tilt_surface" name="camera" use_nominal_extrinsics="true">
     <origin xyz="0 0 0.05" rpy="0 0 0"/>
   </xacro:sensor_d435>

Commit message: fix: align robot geometry with physical image

File: src/dual_arm_torso/urdf/dual_arm_torso.urdf.xacro (robot description, xacro)
@@ -59,5 +59,5 @@
       <!-- The STL X range is -309 to +257. Let's put left carriage at X=-200, Y=100 -->
       <!-- We might need to rotate it if it faces the wrong way. -->
-      <origin xyz="-0.150 0.284 0.050" rpy="0 0 0"/>
+      <origin xyz="-0.086 0.265 0.050" rpy="0 0 0"/>
       <axis xyz="0 0 1"/>
       <limit lower="0.05" upper="0.8" effort="100.0" velocity="0.5"/>
@@ -89,5 +89,5 @@
       <child link="right_carriage_link"/>
       <!-- Estimated position of the right rail. -->
-      <origin xyz="0.150 0.284 0.050" rpy="0 0 0"/>
+      <origin xyz="0.035 0.022 0.050" rpy="0 0 3.14159"/>
       <axis xyz="0 0 1"/>
       <limit lower="0.05" upper="0.8" effort="100.0" velocity="0.5"/>

File: src/pas_dual_arm_bringup/urdf/robot.urdf.xacro (robot description, xacro)
@@ -13,5 +13,5 @@
        Let's place it at the center of the base, somewhat elevated. -->
   <xacro:dual_arm_torso parent="base_footprint">
-    <origin xyz="0 0 0.2" rpy="0 0 -1.5708"/>
+    <origin xyz="0 0 0.2" rpy="0 0 0"/>
   </xacro:dual_arm_torso>
   <!-- 3. KINOVA GEN3 ARMS -->
@@ -34,5 +34,5 @@
     connection_inactivity_timeout_ms="2000"
     sim_ignition="$(arg sim_ignition)">
-    <origin xyz="0.060 0.047 0.112" rpy="-1.5708 0 0"/>
+    <origin xyz="0.060 0.0735 0.112" rpy="-1.5708 0 0"/>
   </xacro:load_robot>
   <!-- Right Arm -->
@@ -53,5 +53,5 @@
     connection_inactivity_timeout_ms="2000"
     sim_ignition="$(arg sim_ignition)">
-    <origin xyz="0.060 0.047 0.112" rpy="-1.5708 0 0"/>
+    <origin xyz="0.060 0.0735 0.112" rpy="-1.5708 0 0"/>
   </xacro:load_robot>
   <!-- 4. PAN-TILT & REALSENSE -->
@@ -60,5 +60,5 @@
   <xacro:pan_tilt parent="torso_base_link">
     <!-- Place the pan-tilt at the top of the torso (Z=0.956) -->
-    <origin xyz="0 0 0.956" rpy="0 0 1.5708"/>
+    <origin xyz="0 0 0.956" rpy="0 0 0"/>
   </xacro:pan_tilt>
   <!-- Include Realsense D435 camera URDF -->

Commit message: fix: center torso, inset carriages, and add 45-deg wedge mounts for arms

File: src/dual_arm_torso/urdf/dual_arm_torso.urdf.xacro (robot description, xacro)
@@ -59,5 +59,5 @@
       <!-- The STL X range is -309 to +257. Let's put left carriage at X=-200, Y=100 -->
       <!-- We might need to rotate it if it faces the wrong way. -->
-      <origin xyz="-0.086 0.265 0.050" rpy="0 0 0"/>
+      <origin xyz="-0.086 0.1625 0.050" rpy="0 0 0"/>
       <axis xyz="0 0 1"/>
       <limit lower="0.05" upper="0.8" effort="100.0" velocity="0.5"/>
@@ -89,8 +89,53 @@
       <child link="right_carriage_link"/>
       <!-- Estimated position of the right rail. -->
-      <origin xyz="0.035 0.022 0.050" rpy="0 0 3.14159"/>
+      <origin xyz="0.035 0.1235 0.050" rpy="0 0 3.14159"/>
       <axis xyz="0 0 1"/>
       <limit lower="0.05" upper="0.8" effort="100.0" velocity="0.5"/>
     </joint>
+    <!-- ================== WEDGES ================== -->
+    <link name="left_wedge_link">
+      <visual>
+        <origin xyz="0.060 0 -0.060" rpy="0 0 1.5708"/>
+        <geometry>
+          <mesh filename="package://dual_arm_torso/meshes/wedge.stl" scale="0.001 0.001 0.001"/>
+        </geometry>
+        <material name="wedge_blue">
+          <color rgba="0.1 0.3 0.8 1.0"/>
+        </material>
+      </visual>
+      <collision>
+        <origin xyz="0.060 0 -0.060" rpy="0 0 1.5708"/>
+        <geometry>
+          <mesh filename="package://dual_arm_torso/meshes/wedge.stl" scale="0.001 0.001 0.001"/>
+        </geometry>
+      </collision>
+    </link>
+    <joint name="left_carriage_to_wedge" type="fixed">
+      <parent link="left_carriage_link"/>
+      <child link="left_wedge_link"/>
+      <origin xyz="0.060 0.0735 0.112" rpy="0 0 0"/>
+    </joint>
+    <link name="right_wedge_link">
+      <visual>
+        <origin xyz="0.060 0 -0.060" rpy="0 0 1.5708"/>
+        <geometry>
+          <mesh filename="package://dual_arm_torso/meshes/wedge.stl" scale="0.001 0.001 0.001"/>
+        </geometry>
+        <material name="wedge_blue">
+          <color rgba="0.1 0.3 0.8 1.0"/>
+        </material>
+      </visual>
+      <collision>
+        <origin xyz="0.060 0 -0.060" rpy="0 0 1.5708"/>
+        <geometry>
+          <mesh filename="package://dual_arm_torso/meshes/wedge.stl" scale="0.001 0.001 0.001"/>
+        </geometry>
+      </collision>
+    </link>
+    <joint name="right_carriage_to_wedge" type="fixed">
+      <parent link="right_carriage_link"/>
+      <child link="right_wedge_link"/>
+      <origin xyz="0.060 0.0735 0.112" rpy="0 0 0"/>
+    </joint>
   </xacro:macro>
 </robot>

File: src/pas_dual_arm_bringup/urdf/robot.urdf.xacro (robot description, xacro)
@@ -13,5 +13,5 @@
        Let's place it at the center of the base, somewhat elevated. -->
   <xacro:dual_arm_torso parent="base_footprint">
-    <origin xyz="0 0 0.2" rpy="0 0 0"/>
+    <origin xyz="0.026 -0.143 0.2" rpy="0 0 0"/>
   </xacro:dual_arm_torso>
   <!-- 3. KINOVA GEN3 ARMS -->
@@ -19,5 +19,5 @@
   <!-- Left Arm -->
   <xacro:load_robot
-    parent="left_carriage_link"
+    parent="left_wedge_link"
     prefix="left_"
     arm="gen3"
@@ -34,9 +34,9 @@
     connection_inactivity_timeout_ms="2000"
     sim_ignition="$(arg sim_ignition)">
-    <origin xyz="0.060 0.0735 0.112" rpy="-1.5708 0 0"/>
+    <origin xyz="0 0.060 0" rpy="-0.785398 0 0"/>
   </xacro:load_robot>
   <!-- Right Arm -->
   <xacro:load_robot
-    parent="right_carriage_link"
+    parent="right_wedge_link"
     prefix="right_"
     arm="gen3"
@@ -53,5 +53,5 @@
     connection_inactivity_timeout_ms="2000"
     sim_ignition="$(arg sim_ignition)">
-    <origin xyz="0.060 0.0735 0.112" rpy="-1.5708 0 0"/>
+    <origin xyz="0 0.060 0" rpy="0.785398 0 3.14159"/>
   </xacro:load_robot>
   <!-- 4. PAN-TILT & REALSENSE -->
