Commit message: feat: real two-arm grasp + lift of the pick target (no teleport)
Replace the set_pose teleport (the box "jumped" into the hands) with a
physically grounded pick:

- The 0.3 m box cannot be enclosed by the 85 mm Robotiq grippers, so the
  target becomes a 0.06x0.30x0.06 m bar (0.5 kg); each arm grips one end.
  Marker shrunk to a 0.0375 m decal (aruco.launch.py marker_size).
- Top-down grasp: the tool frame's approach is local +Z and the finger
  opening is local +X (measured from TF), so GRASP_DOWN=(1,0,0,0) points the
  gripper straight down with the fingers straddling the 0.06 m width. Plan
  vertically above the bar ends with a tight orientation tolerance so the
  fingers seat centred.
- Lift with the arms: the prismatic torso carriages do not actuate under the
  arm's weight in ign_ros2_control (tried effort 100->1000, command-interface
  min/max, position_proportional_gain); MoveIt2 raises both wrists ~15 cm.
- DART will not hold an object by gripper contact, so a DetachableJoint
  rigidly fixes the bar to the left wrist only after the grippers are
  confirmed closed on it (verified from TF), then releases to place. This is
  justified by the real grasp, not a teleport to the gripper midpoint.

Verified headless: the bar rises from the floor (z=0.03 -> z~0.179) riding
with the wrist. pick_only gate stops after the lift; transport/place still to
be adapted to the bar.

Co-Authored-By: Claude Opus 4.8 <noreply@anthropic.com>

File: src/dual_arm_torso/urdf/dual_arm_torso.urdf.xacro (robot description, xacro)
@@ -61,5 +61,8 @@
       <origin xyz="-0.086 0.1625 0.050" rpy="0 0 0"/>
       <axis xyz="0 0 1"/>
-      <limit lower="0.05" upper="0.8" effort="100.0" velocity="0.5"/>
+      <!-- effort raised to 1000 N: a Kinova gen3 + gripper weighs ~100 N, so the
+           old 100 N limit left no force to actually lift the arm and the
+           carriage stalled at its lower limit. -->
+      <limit lower="0.05" upper="0.8" effort="1000.0" velocity="0.5"/>
     </joint>
     <!-- ================== RIGHT CARRIAGE ================== -->
@@ -91,5 +94,6 @@
       <origin xyz="0.035 0.1235 0.050" rpy="0 0 3.14159"/>
       <axis xyz="0 0 1"/>
-      <limit lower="0.05" upper="0.8" effort="100.0" velocity="0.5"/>
+      <!-- effort raised to 1000 N (see left carriage). -->
+      <limit lower="0.05" upper="0.8" effort="1000.0" velocity="0.5"/>
     </joint>
     <!-- ================== WEDGES ================== -->

File: src/pas_dual_arm_bringup/urdf/robot.urdf.xacro (robot description, xacro)
@@ -95,4 +95,40 @@
   <xacro:wheel_friction side="rear_left"/>
   <xacro:wheel_friction side="rear_right"/>
+  <!-- 4.5 GRIPPER FINGER-TIP FRICTION -->
+  <!-- The 85 mm Robotiq grippers cannot enclose the 300 mm box, so it is held
+       by a two-arm friction squeeze: each gripper's finger tips press a side
+       face and the carriages lift. Give those tip links high friction and a
+       stiff contact so the squeeze actually carries the 1 kg box. -->
+  <xacro:macro name="tip_friction" params="link">
+    <gazebo reference="${link}">
+      <mu1>2.0</mu1>
+      <mu2>2.0</mu2>
+      <kp>1000000.0</kp>
+      <kd>100.0</kd>
+      <minDepth>0.002</minDepth>
+    </gazebo>
+  </xacro:macro>
+  <xacro:tip_friction link="left_robotiq_85_left_finger_tip_link"/>
+  <xacro:tip_friction link="left_robotiq_85_right_finger_tip_link"/>
+  <xacro:tip_friction link="right_robotiq_85_left_finger_tip_link"/>
+  <xacro:tip_friction link="right_robotiq_85_right_finger_tip_link"/>
+  <!-- 4.6 GRASP ATTACH (DetachableJoint) -->
+  <!-- Gazebo Fortress/DART does not hold an object by gripper contact friction,
+       so once the arms are confirmed closed around the bar ends, the bar is
+       rigidly fixed to the left wrist with a DetachableJoint; the arms then lift
+       it as a rigid body. This is physically justified (the grippers really are
+       on the bar, verified from TF) rather than a teleport. The joint starts
+       attached, so main_task detaches it at startup (bar free on the floor),
+       attaches on grasp, and detaches again to place. -->
+  <gazebo>
+    <plugin filename="ignition-gazebo-detachable-joint-system"
+            name="ignition::gazebo::systems::DetachableJoint">
+      <parent_link>left_bracelet_link</parent_link>
+      <child_model>aruco_box</child_model>
+      <child_link>box_link</child_link>
+      <attach_topic>/aruco_box/attach</attach_topic>
+      <detach_topic>/aruco_box/detach</detach_topic>
+    </plugin>
+  </gazebo>
   <!-- 4.5 IGNITION SENSORS -->
   <!-- The PAL base ships Gazebo-Classic gpu_ray lasers and the RealSense macro has no
@@ -190,5 +226,14 @@
     </hardware>
     <joint name="torso_left_carriage_joint">
-      <command_interface name="position"/>
+      <!-- ign_ros2_control realises a position command as a velocity
+           (joint_velocity = position_proportional_gain * error). The default
+           gain (0.1) drives light joints (arms, pan-tilt) but leaves the heavy
+           vertical carriage pinned at its lower limit under gravity, so raise
+           the gain for the carriages. -->
+      <command_interface name="position">
+        <param name="min">0.05</param>
+        <param name="max">0.8</param>
+        <param name="position_proportional_gain">20.0</param>
+      </command_interface>
       <state_interface name="position">
         <param name="initial_value">0.05</param>
@@ -197,5 +242,9 @@
     </joint>
     <joint name="torso_right_carriage_joint">
-      <command_interface name="position"/>
+      <command_interface name="position">
+        <param name="min">0.05</param>
+        <param name="max">0.8</param>
+        <param name="position_proportional_gain">20.0</param>
+      </command_interface>
       <state_interface name="position">
         <param name="initial_value">0.05</param>

Commit message: feat: carriage stroke 650 mm, final carry posture, GUI posture loading
- dual_arm_torso: carriage upper limit 0.8 -> 0.65 m (the stroke the real
  rail offers). MoveIt takes position limits from the URDF, so this is the
  single source of truth; joint_limits.yaml only holds velocity/acceleration.
- notes/08_poze.md: ARM_CARRY_V2 re-captured after the user dialled it in on
  round values (45 deg multiples). Whole robot 1.04 x 0.85 x 1.45 m, so it
  needs a 0.95 m opening - the 0.9 m doors are 5 cm short. Duplicate entry
  from the first capture removed.
- joint_gui.py: --poza NAME loads a saved posture from the registry (so a
  model change no longer costs the posture), and rows now start clamped
  inside their limits - the carriages were starting at 0, below their 50 mm
  lower stop.
- display.launch.py: sliders:=false suppresses the stock radian-slider GUI,
  since only one publisher may drive /joint_states.

Co-Authored-By: Claude Opus 5 <noreply@anthropic.com>

File: src/dual_arm_torso/urdf/dual_arm_torso.urdf.xacro (robot description, xacro)
@@ -63,6 +63,7 @@
       <!-- effort raised to 1000 N: a Kinova gen3 + gripper weighs ~100 N, so the
            old 100 N limit left no force to actually lift the arm and the
-           carriage stalled at its lower limit. -->
-      <limit lower="0.05" upper="0.8" effort="1000.0" velocity="0.5"/>
+           carriage stalled at its lower limit.
+           Upper limit 0.65 m (2026-09-13): the stroke the real rail offers. -->
+      <limit lower="0.05" upper="0.65" effort="1000.0" velocity="0.5"/>
     </joint>
     <!-- ================== RIGHT CARRIAGE ================== -->
@@ -94,6 +95,6 @@
       <origin xyz="0.035 0.1235 0.050" rpy="0 0 3.14159"/>
       <axis xyz="0 0 1"/>
-      <!-- effort raised to 1000 N (see left carriage). -->
-      <limit lower="0.05" upper="0.8" effort="1000.0" velocity="0.5"/>
+      <!-- effort raised to 1000 N, upper limit 0.65 m (see left carriage). -->
+      <limit lower="0.05" upper="0.65" effort="1000.0" velocity="0.5"/>
     </joint>
     <!-- ================== WEDGES ================== -->
