Commit message: fix: convert wedge STL to binary, adjust torso height, and fix pan-tilt/camera mounting

File: src/pas_dual_arm_bringup/urdf/robot.urdf.xacro (robot description, xacro)
@@ -13,5 +13,5 @@
        Let's place it at the center of the base, somewhat elevated. -->
   <xacro:dual_arm_torso parent="base_footprint">
-    <origin xyz="0.026 -0.143 0.2" rpy="0 0 0"/>
+    <origin xyz="0.026 -0.143 0.31" rpy="0 0 0"/>
   </xacro:dual_arm_torso>
   <!-- 3. KINOVA GEN3 ARMS -->
@@ -59,6 +59,6 @@
   <xacro:include filename="$(find pan_tilt_description)/urdf/pan_tilt.urdf.xacro"/>
   <xacro:pan_tilt parent="torso_base_link">
-    <!-- Place the pan-tilt at the top of the torso (Z=0.956) -->
-    <origin xyz="0 0 0.956" rpy="0 0 0"/>
+    <!-- Place the pan-tilt at the center of the front beam -->
+    <origin xyz="0.237 0.143 0.956" rpy="0 0 0"/>
   </xacro:pan_tilt>
   <!-- Include Realsense D435 camera URDF -->
@@ -67,5 +67,5 @@
   <!-- Attach the camera to the pan_tilt top link -->
   <xacro:sensor_d435 parent="pan_tilt_surface" name="camera" use_nominal_extrinsics="true">
-    <origin xyz="0 0 0.05" rpy="0 0 0"/>
+    <origin xyz="0 0 0" rpy="0 0 0"/>
   </xacro:sensor_d435>
   <!-- 5. ROS2_CONTROL & GAZEBO IGNITION PLUGIN -->

Commit message: feat: complete visual geometry and scale calibration of PAS dual arm robot

File: src/pas_dual_arm_bringup/urdf/robot.urdf.xacro (robot description, xacro)
@@ -59,6 +59,6 @@
   <xacro:include filename="$(find pan_tilt_description)/urdf/pan_tilt.urdf.xacro"/>
   <xacro:pan_tilt parent="torso_base_link">
-    <!-- Place the pan-tilt at the center of the front beam -->
-    <origin xyz="0.237 0.143 0.956" rpy="0 0 0"/>
+    <!-- Place the pan-tilt on the front beam (moved back to sit on the beam) -->
+    <origin xyz="0.060 0.143 0.956" rpy="0 0 0"/>
   </xacro:pan_tilt>
   <!-- Include Realsense D435 camera URDF -->
