Commit message: feat: working ros2_control in Gazebo Fortress + reliable launch (M0+M1)
M0 - reliable launch:
- Force Fast DDS in sim/display/nav2 launches (the global rmw_zenoh override in
  ~/.bashrc points at an unreachable router and crashes every node locally).
- Fix sim.launch.py robot_description (wrap xacro Command in ParameterValue);
  it was being parsed as YAML, so the Gazebo sim never actually launched before.

M1 - controllers active in Gazebo:
- Bypass PAL omni_base ros2_control (targets Gazebo Classic GazeboSystem, which
  ign_ros2_control cannot load); drive the base with the Ignition MecanumDrive
  system plugin via /cmd_vel (+ /odom + TF) instead.
- Add ign_ros2_control blocks for the torso prismatic carriages and the pan-tilt
  joints (previously had no command interfaces).
- Rewrite controllers.yaml with real joint lists: left/right arm + torso + pan-tilt
  JointTrajectoryControllers and left/right GripperActionControllers.
- Spawn all controllers from sim.launch.py with a large CM timeout.

Verified live: model loads with 0 urdf2sdf errors, controller_manager up with all
7 controllers active, commanded left_joint_2 -> 0.8 and it reached 0.799.

Co-Authored-By: Claude Opus 4.8 <noreply@anthropic.com>

File: src/pas_dual_arm_bringup/urdf/robot.urdf.xacro (robot description, xacro)
@@ -5,6 +5,15 @@
   <xacro:arg name="sim_ignition" default="true"/>
   <!-- 1. OMNI BASE -->
-  <!-- We include the omni_base description. It provides the base_link and wheels. -->
-  <xacro:include filename="$(find omni_base_description)/robots/omni_base.urdf.xacro"/>
+  <!-- We include ONLY the structural part of the omni_base (base_link, base_footprint,
+       wheels, lasers, imu). We deliberately do NOT include robots/omni_base.urdf.xacro,
+       because it appends a ros2_control block bound to gazebo_ros2_control/GazeboSystem
+       (Gazebo Classic), which the ign_ros2_control plugin cannot load under Fortress.
+       The base is instead driven by the Ignition MecanumDrive plugin (see section 5). -->
+  <xacro:property name="namespace" value=""/>
+  <xacro:property name="is_public_sim" value="true"/>
+  <xacro:include filename="$(find pal_urdf_utils)/urdf/materials.urdf.xacro"/>
+  <xacro:include filename="$(find pal_urdf_utils)/urdf/deg_to_rad.urdf.xacro"/>
+  <xacro:include filename="$(find omni_base_description)/urdf/base/base_sensors.urdf.xacro"/>
+  <xacro:base_sensors name="base" front_laser_model="sick-571" rear_laser_model="sick-571"/>
   <!-- 2. DUAL ARM TORSO -->
   <!-- We include our custom torso and attach it to the base_link -->
@@ -69,9 +78,70 @@
     <origin xyz="0 0 0" rpy="0 0 0"/>
   </xacro:sensor_d435>
-  <!-- 5. ROS2_CONTROL & GAZEBO IGNITION PLUGIN -->
+  <!-- 5. ROS2_CONTROL FOR TORSO AND PAN-TILT -->
+  <!-- The Kinova arms and Robotiq grippers already declare their own
+       ign_ros2_control blocks (via load_robot, sim_ignition:=true). The custom torso
+       carriages and the pan-tilt joints do not, so we declare them here. -->
+  <ros2_control name="torso_system" type="system">
+    <hardware>
+      <plugin>ign_ros2_control/IgnitionSystem</plugin>
+    </hardware>
+    <joint name="torso_left_carriage_joint">
+      <command_interface name="position"/>
+      <state_interface name="position">
+        <param name="initial_value">0.05</param>
+      </state_interface>
+      <state_interface name="velocity"/>
+    </joint>
+    <joint name="torso_right_carriage_joint">
+      <command_interface name="position"/>
+      <state_interface name="position">
+        <param name="initial_value">0.05</param>
+      </state_interface>
+      <state_interface name="velocity"/>
+    </joint>
+  </ros2_control>
+  <ros2_control name="pan_tilt_system" type="system">
+    <hardware>
+      <plugin>ign_ros2_control/IgnitionSystem</plugin>
+    </hardware>
+    <joint name="pan_tilt_yaw_joint">
+      <command_interface name="position"/>
+      <state_interface name="position">
+        <param name="initial_value">0.0</param>
+      </state_interface>
+      <state_interface name="velocity"/>
+    </joint>
+    <joint name="pan_tilt_pitch_joint">
+      <command_interface name="position"/>
+      <state_interface name="position">
+        <param name="initial_value">0.0</param>
+      </state_interface>
+      <state_interface name="velocity"/>
+    </joint>
+  </ros2_control>
+  <!-- 6. IGNITION SYSTEM PLUGINS -->
   <gazebo>
+    <!-- ros2_control manager: loads ALL ros2_control blocks (arms, grippers, torso, pan-tilt) -->
     <plugin filename="ign_ros2_control-system" name="ign_ros2_control::IgnitionROS2ControlPlugin">
       <parameters>$(find pas_dual_arm_bringup)/config/controllers.yaml</parameters>
     </plugin>
+    <!-- Omnidirectional base drive (replaces PAL's Gazebo-Classic planar_move).
+         Subscribes to /cmd_vel (Twist) and publishes /odom + odom->base_footprint TF. -->
+    <plugin filename="ignition-gazebo-mecanum-drive-system"
+            name="ignition::gazebo::systems::MecanumDrive">
+      <front_left_joint>wheel_front_left_joint</front_left_joint>
+      <front_right_joint>wheel_front_right_joint</front_right_joint>
+      <back_left_joint>wheel_rear_left_joint</back_left_joint>
+      <back_right_joint>wheel_rear_right_joint</back_right_joint>
+      <wheel_separation>0.44715</wheel_separation>
+      <wheelbase>0.488</wheelbase>
+      <wheel_radius>0.0762</wheel_radius>
+      <topic>cmd_vel</topic>
+      <odom_topic>odom</odom_topic>
+      <tf_topic>tf</tf_topic>
+      <frame_id>odom</frame_id>
+      <child_frame_id>base_footprint</child_frame_id>
+      <odom_publish_frequency>50</odom_publish_frequency>
+    </plugin>
   </gazebo>
 </robot>

Commit message: feat: Nav2 autonomous navigation with diff_drive base (M5)
Drive the omni_base through ros2_control + diff_drive_controller (PAL's
Classic planar_move never instantiates on Fortress), giving x+yaw motion,
wheel-encoder odometry and odom->base_footprint TF.

- urdf: ros2_control velocity system for the 4 base wheels + friction
  override (PAL zeroes wheel mu for their kinematic sim).
- controllers.yaml: base_controller (diff_drive_controller) config.
- nav2_params.yaml: slam_toolbox + Nav2 (NavFn planner, DWB controller),
  costmaps from /scan, footprint/frames for this robot.
- nav2.launch.py: slam + Nav2, Nav2 delayed via TimerAction so SLAM
  publishes map->odom first.
- cmd_vel_relay: bridges Nav2 /cmd_vel -> /base_controller/cmd_vel_unstamped
  (controller lives inside the gz controller_manager, so no plain remap).

Verified live: full TF chain map->odom->base_footprint->base_link, goal
sent on /goal_pose produces non-zero /cmd_vel and the base physically
drives toward it (odom x 0 -> 0.24 m).

Co-Authored-By: Claude Fable 5 <noreply@anthropic.com>

File: src/pas_dual_arm_bringup/urdf/robot.urdf.xacro (robot description, xacro)
@@ -78,4 +78,21 @@
     <origin xyz="0 0 0" rpy="0 0 0"/>
   </xacro:sensor_d435>
+  <!-- 4.4 WHEEL FRICTION OVERRIDE -->
+  <!-- PAL's wheel.gazebo.xacro sets mu1=mu2=0.0 on every wheel (their Classic sim
+       drives the base kinematically with planar_move, so wheels are decorative).
+       Our diff_drive base actually rolls on the wheels, so give them traction. -->
+  <xacro:macro name="wheel_friction" params="side">
+    <gazebo reference="wheel_${side}_link">
+      <mu1>1.5</mu1>
+      <mu2>1.5</mu2>
+      <kp>1000000.0</kp>
+      <kd>1000.0</kd>
+      <minDepth>0.003</minDepth>
+    </gazebo>
+  </xacro:macro>
+  <xacro:wheel_friction side="front_left"/>
+  <xacro:wheel_friction side="front_right"/>
+  <xacro:wheel_friction side="rear_left"/>
+  <xacro:wheel_friction side="rear_right"/>
   <!-- 4.5 IGNITION SENSORS -->
   <!-- The PAL base ships Gazebo-Classic gpu_ray lasers and the RealSense macro has no
@@ -138,4 +155,34 @@
        ign_ros2_control blocks (via load_robot, sim_ignition:=true). The custom torso
        carriages and the pan-tilt joints do not, so we declare them here. -->
+  <!-- Wheel drive through ros2_control (velocity interfaces) + diff_drive_controller.
+       The PAL ros2_control block targets Gazebo Classic and the Fortress built-in
+       drive systems (MecanumDrive/VelocityControl) never instantiate on this
+       install, while gz_ros2_control demonstrably works - so the wheels are driven
+       the same way as every other joint of this robot. -->
+  <ros2_control name="base_wheels_system" type="system">
+    <hardware>
+      <plugin>ign_ros2_control/IgnitionSystem</plugin>
+    </hardware>
+    <joint name="wheel_front_left_joint">
+      <command_interface name="velocity"/>
+      <state_interface name="position"/>
+      <state_interface name="velocity"/>
+    </joint>
+    <joint name="wheel_front_right_joint">
+      <command_interface name="velocity"/>
+      <state_interface name="position"/>
+      <state_interface name="velocity"/>
+    </joint>
+    <joint name="wheel_rear_left_joint">
+      <command_interface name="velocity"/>
+      <state_interface name="position"/>
+      <state_interface name="velocity"/>
+    </joint>
+    <joint name="wheel_rear_right_joint">
+      <command_interface name="velocity"/>
+      <state_interface name="position"/>
+      <state_interface name="velocity"/>
+    </joint>
+  </ros2_control>
   <ros2_control name="torso_system" type="system">
     <hardware>
@@ -182,22 +229,8 @@
       <parameters>$(find pas_dual_arm_bringup)/config/controllers.yaml</parameters>
     </plugin>
-    <!-- Omnidirectional base drive (replaces PAL's Gazebo-Classic planar_move).
-         Subscribes to /cmd_vel (Twist) and publishes /odom + odom->base_footprint TF. -->
-    <plugin filename="ignition-gazebo-mecanum-drive-system"
-            name="ignition::gazebo::systems::MecanumDrive">
-      <front_left_joint>wheel_front_left_joint</front_left_joint>
-      <front_right_joint>wheel_front_right_joint</front_right_joint>
-      <back_left_joint>wheel_rear_left_joint</back_left_joint>
-      <back_right_joint>wheel_rear_right_joint</back_right_joint>
-      <wheel_separation>0.44715</wheel_separation>
-      <wheelbase>0.488</wheelbase>
-      <wheel_radius>0.0762</wheel_radius>
-      <topic>cmd_vel</topic>
-      <odom_topic>odom</odom_topic>
-      <tf_topic>tf</tf_topic>
-      <frame_id>odom</frame_id>
-      <child_frame_id>base_footprint</child_frame_id>
-      <odom_publish_frequency>50</odom_publish_frequency>
-    </plugin>
+    <!-- Base motion + odometry are handled by the ros2_control diff_drive
+         base_controller (see base_wheels_system above and controllers.yaml).
+         The Fortress built-in drive systems (MecanumDrive, VelocityControl) were
+         tried first but never instantiate on this install. -->
   </gazebo>
 </robot>

Commit message: feat: assignment cube (0.3m/1kg) + verified dual-arm squeeze grasp+lift
The world now carries the ASSIGNMENT box (0.3x0.3x0.3 m, 1 kg cube) instead
of the graspable slab workaround. Since the 85 mm grippers cannot enclose a
0.3 m face, both arms press opposite side faces with their CLOSED grippers
(fingertip pads carry gz Contact sensors) and the DetachableJoint attach is
committed only after box-only contact is proven on BOTH pads plus an
independent fingertip-geometry check. 3 full grasp+lift cycles verified in
the GUI; every failed attempt aborted honestly (no fake attach).

Highlights (details in STATE.md):
- measure BEFORE close-in (self-in-view junk clusters), odometry-corrected
  drive, sim-time cmd_vel pacing (RTF<1 halved every open-loop distance)
- asymmetric centering turn (arms' feasible press regions do not overlap)
- planning scene obstacles (floor/table/cube) - RRT no longer sweeps arms
  through the table
- press as straight Cartesian line executed on BOTH arm controllers
  simultaneously (lone press bulldozes the cube), with time
  parameterization, 2*pi unwrap (the 'weird full-turn rotations'),
  stale-start guard, settle-waits and a near-face RRT + re-press fallback
- contact sensors bridged from the real Fortress per-sensor topics
  (custom <topic> tag is ignored) and gated to aruco_box collisions only
- env fixes: gazebo_version xacro property (pal_urdf_utils update),
  geometric_shapes ABI compat for the ws_moveit2 source build

Known gap: the final lowering can release the cube a few cm high (tips
over); transport to the second room remains open (Phase 1/3 in STATE.md).

Co-Authored-By: Claude Fable 5 <noreply@anthropic.com>

File: src/pas_dual_arm_bringup/urdf/robot.urdf.xacro (robot description, xacro)
@@ -12,4 +12,8 @@
   <xacro:property name="namespace" value=""/>
   <xacro:property name="is_public_sim" value="true"/>
+  <!-- pal_urdf_utils laser/sensor macros branch on this; we skip omni_base.urdf.xacro
+       (see note above) so it's never set upstream. Anything != 'classic' is correct
+       here since we run on Ignition/gz sim, not Gazebo Classic. -->
+  <xacro:property name="gazebo_version" value="gazebo"/>
   <xacro:include filename="$(find pal_urdf_utils)/urdf/materials.urdf.xacro"/>
   <xacro:include filename="$(find pal_urdf_utils)/urdf/deg_to_rad.urdf.xacro"/>
@@ -121,4 +125,31 @@
   <xacro:tip_friction link="right_robotiq_85_left_finger_link"/>
   <xacro:tip_friction link="right_robotiq_85_right_finger_link"/>
+  <!-- 4.5b FINGER-TIP CONTACT SENSORS -->
+  <!-- Ignition contact sensor on each finger tip so the grasp is confirmed by a
+       REAL finger-on-box contact ("small contact force"), not by geometry alone.
+       main_task fuses these with the depth check and the gripper stall before it
+       commits the rigid attach. The collision name is sdformat's default for an
+       unnamed URDF collision: <link>_collision. Needs the world's Contact system
+       plugin. If a sensor never fires, the grasp still verifies via depth+stall. -->
+  <xacro:macro name="tip_contact" params="link sensor topic">
+    <gazebo reference="${link}">
+      <sensor name="${sensor}" type="contact">
+        <always_on>1</always_on>
+        <update_rate>50</update_rate>
+        <contact>
+          <collision>${link}_collision</collision>
+        </contact>
+        <topic>${topic}</topic>
+      </sensor>
+    </gazebo>
+  </xacro:macro>
+  <xacro:tip_contact link="left_robotiq_85_left_finger_tip_link"
+                     sensor="left_left_tip_contact" topic="/contact/left_left_tip"/>
+  <xacro:tip_contact link="left_robotiq_85_right_finger_tip_link"
+                     sensor="left_right_tip_contact" topic="/contact/left_right_tip"/>
+  <xacro:tip_contact link="right_robotiq_85_left_finger_tip_link"
+                     sensor="right_left_tip_contact" topic="/contact/right_left_tip"/>
+  <xacro:tip_contact link="right_robotiq_85_right_finger_tip_link"
+                     sensor="right_right_tip_contact" topic="/contact/right_right_tip"/>
   <!-- 4.6 CONTACT-VERIFIED GRASP ATTACH (DetachableJoint) -->
   <!-- DART will not hold a free object by gripper friction (tried mu up to 5,

Commit message: checkpoint: mapping and localization stack as it stood after run 44
Brings the whole SLAM/localization surface under version control before the
navigation work starts, so there is a point to return to.

- slam_toolbox config, mapping launch, scan self-filter, mapping tour
- accepted map (seminar_map.yaml/.pgm) and the hand-written keepout mask
- posture registry, base drive mixin, feature registry, go_to_room
- mecanum base controller, split base URDF, AMCL/Nav2 params
- notes: run log through run 44, P-37/P-38, workspace debug survey, runbook

Map pose graphs (.posegraph/.data, ~16 MB per map) and timestamped archives
stay out of git; only the .yaml/.pgm pair map_server needs is tracked.

Co-Authored-By: Claude Opus 5 <noreply@anthropic.com>

File: src/pas_dual_arm_bringup/urdf/robot.urdf.xacro (robot description, xacro)
@@ -1,7 +1,10 @@
-<?xml version="1.0"?>
-<robot xmlns:xacro="http://ros.org/wiki/xacro" name="dual_arm_robot">
+<robot xmlns:xacro="http://ros.org/wiki/xacro"
+       xmlns:ignition="http://ignitionrobotics.org/schema"
+       xmlns:gz="http://gazebosim.org/schema"
+       name="dual_arm_robot">
   <!-- Arguments -->
   <xacro:arg name="use_sim_time" default="true"/>
   <xacro:arg name="sim_ignition" default="true"/>
+  <xacro:arg name="carry_arms" default="false"/>
   <!-- 1. OMNI BASE -->
   <!-- We include ONLY the structural part of the omni_base (base_link, base_footprint,
@@ -18,6 +21,13 @@
   <xacro:include filename="$(find pal_urdf_utils)/urdf/materials.urdf.xacro"/>
   <xacro:include filename="$(find pal_urdf_utils)/urdf/deg_to_rad.urdf.xacro"/>
-  <xacro:include filename="$(find omni_base_description)/urdf/base/base_sensors.urdf.xacro"/>
-  <xacro:base_sensors name="base" front_laser_model="sick-571" rear_laser_model="sick-571"/>
+  <xacro:include filename="$(find pas_dual_arm_bringup)/urdf/base/base_sensors.urdf.xacro"/>
+  <!-- Both PAL SICK lasers are disabled on purpose. They are Gazebo-Classic gpu_ray
+       sensors, so they publish nothing under Fortress (see section 6), yet their meshes
+       sit at (+-0.27512, -+0.18297, 0.13244) - exactly in the scan plane of the 360 deg
+       gpu_lidar we mount on virtual_base_laser_link. They showed up as two 7-ray blobs at
+       ~0.31 m in every scan, which would smear into the SLAM map as obstacles that travel
+       with the robot. Disabling them keeps virtual_base_laser_link, which the macro
+       creates unconditionally. -->
+  <xacro:base_sensors name="base" front_laser_model="false" rear_laser_model="false"/>
   <!-- 2. DUAL ARM TORSO -->
   <!-- We include our custom torso and attach it to the base_link -->
@@ -30,4 +40,13 @@
   <!-- 3. KINOVA GEN3 ARMS -->
   <xacro:include filename="$(find kortex_description)/robots/kortex_robot.xacro"/>
+  <!-- Mapping starts in the existing measured carry posture. This avoids a
+       large arm sweep that destabilizes the Fortress/DART simulation. The
+       standard task spawn remains unchanged unless explicitly requested. -->
+  <xacro:property name="initial_left_arm" value="${dict(joint_1=0.0,joint_2=0.0,joint_3=0.0,joint_4=0.0,joint_5=0.0,joint_6=0.0,joint_7=0.0)}"/>
+  <xacro:property name="initial_right_arm" value="${dict(joint_1=0.0,joint_2=0.0,joint_3=0.0,joint_4=0.0,joint_5=0.0,joint_6=0.0,joint_7=0.0)}"/>
+  <xacro:if value="$(arg carry_arms)">
+    <xacro:property name="initial_left_arm" value="${dict(joint_1=0.0,joint_2=1.571,joint_3=2.356,joint_4=-1.571,joint_5=-0.785,joint_6=1.571,joint_7=1.571)}"/>
+    <xacro:property name="initial_right_arm" value="${dict(joint_1=0.0,joint_2=1.571,joint_3=0.785,joint_4=1.571,joint_5=0.785,joint_6=-1.571,joint_7=-1.571)}"/>
+  </xacro:if>
   <!-- Left Arm -->
   <xacro:load_robot
@@ -46,5 +65,6 @@
     session_inactivity_timeout_ms="60000"
     connection_inactivity_timeout_ms="2000"
-    sim_ignition="$(arg sim_ignition)">
+    sim_ignition="$(arg sim_ignition)"
+    initial_positions="${initial_left_arm}">
     <origin xyz="0 0.060 0" rpy="-0.785398 0 0"/>
   </xacro:load_robot>
@@ -65,5 +85,6 @@
     session_inactivity_timeout_ms="60000"
     connection_inactivity_timeout_ms="2000"
-    sim_ignition="$(arg sim_ignition)">
+    sim_ignition="$(arg sim_ignition)"
+    initial_positions="${initial_right_arm}">
     <origin xyz="0 0.060 0" rpy="0.785398 0 3.14159"/>
   </xacro:load_robot>
@@ -82,25 +103,4 @@
     <origin xyz="0 0 0" rpy="0 0 0"/>
   </xacro:sensor_d435>
-  <!-- 4.4 WHEEL FRICTION OVERRIDE -->
-  <!-- PAL's wheel.gazebo.xacro sets mu1=mu2=0.0 on every wheel (their Classic sim
-       drives the base kinematically with planar_move, so wheels are decorative).
-       Our diff_drive base actually rolls on the wheels, so give them rolling
-       traction (mu1) but LOW lateral friction (mu2): this is a rigid 4-wheel
-       skid-steer, so turning in place needs the wheels to slide sideways. With
-       high mu2 the base could only drive straight and would not rotate at all
-       (the 360 scan and all turns were impossible). -->
-  <xacro:macro name="wheel_friction" params="side">
-    <gazebo reference="wheel_${side}_link">
-      <mu1>0.4</mu1>
-      <mu2>0.0</mu2>
-      <kp>1000000.0</kp>
-      <kd>1000.0</kd>
-      <minDepth>0.003</minDepth>
-    </gazebo>
-  </xacro:macro>
-  <xacro:wheel_friction side="front_left"/>
-  <xacro:wheel_friction side="front_right"/>
-  <xacro:wheel_friction side="rear_left"/>
-  <xacro:wheel_friction side="rear_right"/>
   <!-- 4.5 GRIPPER FINGER-TIP FRICTION -->
   <!-- The 85 mm Robotiq grippers cannot enclose the 300 mm box, so it is held
@@ -168,4 +168,5 @@
       <attach_topic>/aruco_box/attach</attach_topic>
       <detach_topic>/aruco_box/detach</detach_topic>
+      <output_topic>/aruco_box/state</output_topic>
     </plugin>
   </gazebo>
@@ -315,5 +316,5 @@
       <command_interface name="position"/>
       <state_interface name="position">
-        <param name="initial_value">0.0</param>
+        <param name="initial_value">0.45</param>
       </state_interface>
       <state_interface name="velocity"/>
