Commit message: feat: markers on the pressed faces, and wrist cameras to read them
The head camera puts the cube within a couple of centimetres, which is enough
to reach a pre-grasp pose a hand's breadth from each face but not to close that
last stretch: the hands stop where dead reckoning says the face is, and that is
not quite where it is. So give each hand something of its own to look at.

The cube now carries an ArUco marker on each of the two faces that get pressed
- id 1 on the face the left hand takes, id 2 on the right. They are smaller
than the front marker, a 0.12 m plate rather than 0.22 m, because at the range
the hand actually stops at, the big plate overflows the frame.

The wrist cameras needed less than expected: the Kinova description already
carries the Gen3 vision module's frames, already in the optical convention, so
only the Gazebo sensor and the bridge entries were missing. One detector
instance per wrist reads its own marker into its own frame.

The detector's pose topic had to become a parameter - three detectors sharing
one topic would have overwritten each other. It defaults to where the head
detector has always published, so nothing downstream changes.

probe_wrist_markers.py answers the question this rests on before anything is
built on top: with the hands at the pre-grasp poses, does each wrist see its
marker, and where does it put it.

Co-Authored-By: Claude Opus 5 <noreply@anthropic.com>

File: src/pas_dual_arm_bringup/urdf/robot.urdf.xacro (robot description, xacro)
@@ -220,4 +220,37 @@
        camera/points) so the box pose and dimensions can be measured by the
        depth sensor for the grasp plan. -->
+  <!-- Wrist cameras. The Kinova description already carries the Gen3 vision
+       module's frames (`*_camera_color_frame`, already in the optical
+       convention), so only the sensor itself was missing. The head camera puts
+       the cube within a couple of centimetres, which is enough to reach the
+       pre-grasp pose but not to close the last 10 cm onto a face; from the
+       pre-grasp pose each wrist looks straight at the marker on the face its
+       own pads will press. Near clip is 0.02 m because the hand ends up within
+       a hand's breadth of the face. -->
+  <xacro:macro name="wrist_camera" params="side">
+    <gazebo reference="${side}_camera_color_frame">
+      <sensor name="${side}_wrist_camera" type="camera">
+        <topic>wrist_${side}</topic>
+        <update_rate>15</update_rate>
+        <always_on>1</always_on>
+        <visualize>false</visualize>
+        <ignition_frame_id>${side}_camera_color_frame</ignition_frame_id>
+        <camera>
+          <horizontal_fov>1.047</horizontal_fov>
+          <image>
+            <width>640</width>
+            <height>480</height>
+            <format>R8G8B8</format>
+          </image>
+          <clip>
+            <near>0.02</near>
+            <far>5.0</far>
+          </clip>
+        </camera>
+      </sensor>
+    </gazebo>
+  </xacro:macro>
+  <xacro:wrist_camera side="left"/>
+  <xacro:wrist_camera side="right"/>
   <gazebo reference="camera_link">
     <sensor name="rgbd_camera" type="rgbd_camera">

Commit message: fix: point the wrist cameras at what their own hands are about to press
kortex_description carries two mountings for the Gen3 vision module and they
disagree. The real one looks along end_effector +Z, which is the gripper's
approach axis. The simulation branch looks along +Y, and its own comment admits
the sim rotation "might not apply to built in vision module". We were on the
sim frame: at a side-grasp pre-pose, +Y works out to straight up in base_link,
so each wrist camera was pointed at the ceiling and could never have seen the
marker on the face its pads press.

So mount the sensor on a frame that follows the real module - optical z along
the approach axis, at the vision module's own origin - with a matching
body-convention frame for the cloud. Verified against the pre-pose rotation:
the approach axis and the new camera axis both come out as [0, -1, 0] in
base_link, straight at the face.

The wrist sensors are rgbd now rather than plain colour, which is also what the
real module is, so each hand contributes a point cloud; all three are bridged,
restamped, and drawn separately in the view.

Pre-grasp standoff doubled to 0.20 m, measured tip-to-face. At a hand's breadth
the pads crowd the cube and the camera is too close to hold the whole marker.
At a cube range of 0.62 m that pose needs 0.819 m of reach, still inside the
envelope.

Co-Authored-By: Claude Opus 5 <noreply@anthropic.com>

File: src/pas_dual_arm_bringup/urdf/robot.urdf.xacro (robot description, xacro)
@@ -229,11 +229,35 @@
        a hand's breadth of the face. -->
   <xacro:macro name="wrist_camera" params="side">
-    <gazebo reference="${side}_camera_color_frame">
-      <sensor name="${side}_wrist_camera" type="camera">
+    <!-- Aim. kortex_description has two mountings for the vision module and
+         they do not agree: the real one looks along end_effector +Z, which is
+         the gripper's approach axis, while the sim branch looks along +Y - and
+         its own comment says the sim rotation "might not apply to built in
+         vision module". At a side-grasp pre-pose, +Y points straight at the
+         ceiling, so on the sim frame the camera could never see the face its
+         own pads press. Mount on a frame that follows the real module: optical
+         z along the approach axis, at the vision module's own origin. -->
+    <link name="${side}_wrist_cam_optical_frame"/>
+    <joint name="${side}_wrist_cam_optical_joint" type="fixed">
+      <origin rpy="0 0 0" xyz="0 0.05639 0.01305"/>
+      <parent link="${side}_end_effector_link"/>
+      <child link="${side}_wrist_cam_optical_frame"/>
+    </joint>
+    <!-- gz ships cloud data in the sensor BODY convention whatever frame it
+         stamps, so give the cloud somewhere correct to be drawn: x along the
+         view, z up in the image. Same role camera_link plays for the head. -->
+    <link name="${side}_wrist_cam_body_frame"/>
+    <joint name="${side}_wrist_cam_body_joint" type="fixed">
+      <origin rpy="1.5707963267948966 -1.5707963267948966 0"
+              xyz="0 0.05639 0.01305"/>
+      <parent link="${side}_end_effector_link"/>
+      <child link="${side}_wrist_cam_body_frame"/>
+    </joint>
+    <gazebo reference="${side}_wrist_cam_optical_frame">
+      <sensor name="${side}_wrist_camera" type="rgbd_camera">
         <topic>wrist_${side}</topic>
         <update_rate>15</update_rate>
         <always_on>1</always_on>
         <visualize>false</visualize>
-        <ignition_frame_id>${side}_camera_color_frame</ignition_frame_id>
+        <ignition_frame_id>${side}_wrist_cam_optical_frame</ignition_frame_id>
         <camera>
           <horizontal_fov>1.047</horizontal_fov>
@@ -247,4 +271,10 @@
             <far>5.0</far>
           </clip>
+          <depth_camera>
+            <clip>
+              <near>0.02</near>
+              <far>3.0</far>
+            </clip>
+          </depth_camera>
         </camera>
       </sensor>

Commit message: fix: aim the wrist cameras by the axis Gazebo actually uses
The clouds came back as slabs flying off in three directions, and the cause was
my own change before this one. An Ignition camera looks along the +X axis of
the link its sensor is attached to, with +Y left and +Z up - not along z. I had
read the Kinova sim frame by its z axis, concluded it pointed at the ceiling,
and moved the sensor onto a frame whose z was right and whose x was sideways.
So the camera ended up aimed along the gripper's opening direction.

Read by the axis that matters, camera_color_frame was the correct mount all
along: its +X is end_effector +Z, the approach axis, and its +Z is up in the
image. That is the same rule the head camera already follows, hanging on
camera_link rather than on an optical frame. The sensor goes back there, and
the cloud is restamped into that frame, since that is the frame gz emits it in.

What was genuinely missing is a frame to name the image in: the detectors solve
PnP in the optical convention, and no Kinova sim frame is that. Declared one, a
half turn about the approach axis, which is also kortex's own non-sim mounting.

Verified numerically at the left pre-grasp pose: approach axis, camera view
direction and optical z all come out [0, -1, 0] in base_link, and image up is
[0, 0, 1].

The view now also shows both wrist images. If the marker is not in those, the
rest of this approach cannot work, and that is worth seeing directly rather
than inferring from a point cloud.

Co-Authored-By: Claude Opus 5 <noreply@anthropic.com>

File: src/pas_dual_arm_bringup/urdf/robot.urdf.xacro (robot description, xacro)
@@ -229,29 +229,23 @@
        a hand's breadth of the face. -->
   <xacro:macro name="wrist_camera" params="side">
-    <!-- Aim. kortex_description has two mountings for the vision module and
-         they do not agree: the real one looks along end_effector +Z, which is
-         the gripper's approach axis, while the sim branch looks along +Y - and
-         its own comment says the sim rotation "might not apply to built in
-         vision module". At a side-grasp pre-pose, +Y points straight at the
-         ceiling, so on the sim frame the camera could never see the face its
-         own pads press. Mount on a frame that follows the real module: optical
-         z along the approach axis, at the vision module's own origin. -->
+    <!-- Aiming rule: an Ignition camera looks along the +X axis of the link
+         its sensor is attached to, with +Y left and +Z up. That is why the
+         head camera hangs on camera_link (x forward) and not on an optical
+         frame. Checked against the Kinova frames: camera_color_frame's +X is
+         end_effector +Z, which is exactly the gripper's approach axis - so it
+         is already the right mount, and the sensor goes there unchanged.
+         The cloud data comes out in that same frame.
+         What was missing is a frame to NAME the image in. The detectors solve
+         PnP in the optical convention (z along the view, x right, y down), and
+         no Kinova sim frame is that, so declare one: a half turn about the
+         approach axis from the end effector. It matches kortex's own non-sim
+         mounting, which is the real module's orientation. -->
     <link name="${side}_wrist_cam_optical_frame"/>
     <joint name="${side}_wrist_cam_optical_joint" type="fixed">
-      <origin rpy="0 0 0" xyz="0 0.05639 0.01305"/>
+      <origin rpy="0 0 3.14159265358979" xyz="0 0.05639 0.01305"/>
       <parent link="${side}_end_effector_link"/>
       <child link="${side}_wrist_cam_optical_frame"/>
     </joint>
-    <!-- gz ships cloud data in the sensor BODY convention whatever frame it
-         stamps, so give the cloud somewhere correct to be drawn: x along the
-         view, z up in the image. Same role camera_link plays for the head. -->
-    <link name="${side}_wrist_cam_body_frame"/>
-    <joint name="${side}_wrist_cam_body_joint" type="fixed">
-      <origin rpy="1.5707963267948966 -1.5707963267948966 0"
-              xyz="0 0.05639 0.01305"/>
-      <parent link="${side}_end_effector_link"/>
-      <child link="${side}_wrist_cam_body_frame"/>
-    </joint>
-    <gazebo reference="${side}_wrist_cam_optical_frame">
+    <gazebo reference="${side}_camera_color_frame">
       <sensor name="${side}_wrist_camera" type="rgbd_camera">
         <topic>wrist_${side}</topic>

Commit message: feat(grasp): pick the cube through the user's DRIVE/DETECTION/GRASP postures
The mission now drives in DRIVE_V4 (carriages 0.20 m, arms tucked, 0.821 m
wide), locates the cube with the head camera at the dock, raises the
carriages to 0.40 m while the arms swing into DETECTION_V4 (through a point
above it, 10 cm clear of the table), drives in to 0.63 m, reads the side
markers with the wrist cameras, moves to GRASP_V4 and sends both tool tips
straight to the marker centres - a 2 mm touch, no squeeze. With contact on
both hands and both tips within 1 cm it attaches the cube (D-05), lifts
0.15 m, pulls it 15 cm towards the robot (elbows swivelled off the torso,
MoveIt-checked), backs away 0.50 m and lowers the carriages to 0.10 m.
Headless run V5: tips 1.3-4.3 mm from target, cube 0.605 m up in Gazebo,
0.821 m wide throughout; the user's GUI run U2 completed too.

Along the way:
- carriages start at 0.06 m, not on their 0.05 m stop, where Ignition
  froze them in both directions (P-13, open since 30 June);
- {left,right}_tool_tip frame at the centre of the closed pads, 0.127 m
  past end_effector_link, which sits at the gripper base;
- MoveIt scene models the real table (0.8 m top, 4 cm thick, legs);
- pose_studio.launch.py: simulation, RViz and pose windows only, nothing
  moves on its own; joint_gui --sim commands the controllers, jogs the
  hands along axes, swivels the elbow with the hand held, mirrors the
  arms exactly, and a saved-poses window loads and saves postures with
  carriages and grippers;
- kinematics.py: whole-robot FK, left/right mirroring, Jacobian jogging;
  grasp_width.py: grasp width over the whole IK null space (P-43);
- notes: P-43, P-44, runs, parameters, run instructions.

Co-Authored-By: Claude Opus 5 <noreply@anthropic.com>

File: src/pas_dual_arm_bringup/urdf/robot.urdf.xacro (robot description, xacro)
@@ -47,6 +47,8 @@
   <xacro:property name="initial_right_arm" value="${dict(joint_1=0.0,joint_2=0.0,joint_3=0.0,joint_4=0.0,joint_5=0.0,joint_6=0.0,joint_7=0.0)}"/>
   <xacro:if value="$(arg carry_arms)">
-    <xacro:property name="initial_left_arm" value="${dict(joint_1=0.0,joint_2=1.571,joint_3=2.356,joint_4=-1.571,joint_5=-0.785,joint_6=1.571,joint_7=1.571)}"/>
-    <xacro:property name="initial_right_arm" value="${dict(joint_1=0.0,joint_2=1.571,joint_3=0.785,joint_4=1.571,joint_5=0.785,joint_6=-1.571,joint_7=-1.571)}"/>
+    <!-- The drive posture: DRIVE_V4 since 16. 9. (user; postures.py), 0.821 m wide,
+         arms tucked. It was ARM_CARRY_V2 before. -->
+    <xacro:property name="initial_left_arm" value="${dict(joint_1=2.182,joint_2=1.244,joint_3=1.396,joint_4=-2.339,joint_5=0.589,joint_6=-0.755,joint_7=2.635)}"/>
+    <xacro:property name="initial_right_arm" value="${dict(joint_1=-2.255,joint_2=1.203,joint_3=-1.278,joint_4=-2.395,joint_5=-0.504,joint_6=-0.769,joint_7=0.536)}"/>
   </xacro:if>
   <!-- Cube-table staging: the wrists start above the 0.75 m tabletop, so the
@@ -161,4 +163,46 @@
   <xacro:tip_contact link="right_robotiq_85_right_finger_tip_link"
                      sensor="right_right_tip_contact" topic="/contact/right_right_tip"/>
+  <!-- Wrist force-torque sensors: EVALUATION ONLY.
+       The real Gen3 has joint torque sensors, not a wrist FT sensor, so no
+       control code may read these - they exist to give the offline
+       qualification an independent reference for the torque-based force
+       estimate. The Fortress contact sensor turned out to publish contact
+       POINTS only, with empty wrenches, so it cannot serve as that reference
+       (notes/03_problemi/P-42). Mounted on joint 7, the sensor sees everything
+       distal to the wrist; the qualifier compares the CHANGE from its zeroed
+       pre-contact value, so the gripper's own weight cancels. -->
+  <xacro:macro name="wrist_force_torque" params="joint sensor topic">
+    <gazebo reference="${joint}">
+      <sensor name="${sensor}" type="force_torque">
+        <always_on>1</always_on>
+        <update_rate>200</update_rate>
+        <topic>${topic}</topic>
+        <force_torque>
+          <frame>child</frame>
+          <measure_direction>parent_to_child</measure_direction>
+        </force_torque>
+      </sensor>
+    </gazebo>
+  </xacro:macro>
+  <xacro:wrist_force_torque joint="left_joint_7"
+                            sensor="left_wrist_ft" topic="/ft/left_wrist"/>
+  <xacro:wrist_force_torque joint="right_joint_7"
+                            sensor="right_wrist_ft" topic="/ft/right_wrist"/>
+  <!-- 4.5 TOOL TIP. end_effector_link sits at the gripper BASE (robotiq_85_base_link
+       is attached to it with no offset); the pads are further out. tool_tip is the
+       centre of the CLOSED pads (knuckle 0.791, as every V4 posture is saved):
+       0.127 m along the tool axis, measured from the collision meshes (the leading
+       pad edge is at 0.163 m). The grasp targets and reach checks are about this
+       point, not the gripper base. -->
+  <xacro:macro name="tool_tip" params="side">
+    <link name="${side}_tool_tip"/>
+    <joint name="${side}_tool_tip_joint" type="fixed">
+      <parent link="${side}_end_effector_link"/>
+      <child link="${side}_tool_tip"/>
+      <origin xyz="0 0 0.127" rpy="0 0 0"/>
+    </joint>
+  </xacro:macro>
+  <xacro:tool_tip side="left"/>
+  <xacro:tool_tip side="right"/>
   <!-- 4.6 CONTACT-VERIFIED GRASP ATTACH (DetachableJoint) -->
   <!-- DART will not hold a free object by gripper friction (tried mu up to 5,
@@ -343,16 +387,25 @@
     </hardware>
     <joint name="torso_left_carriage_joint">
-      <!-- ign_ros2_control realises a position command as a velocity
-           (joint_velocity = position_proportional_gain * error). The default
-           gain (0.1) drives light joints (arms, pan-tilt) but leaves the heavy
-           vertical carriage pinned at its lower limit under gravity, so raise
-           the gain for the carriages. -->
+      <!-- ign_ros2_control realises a position command as a joint velocity
+           (joint_velocity = position_proportional_gain * error). The gain is a
+           parameter of the PLUGIN'S OWN node, not of a joint: this tag never
+           reached it, every run logged the 0.1 default, and setting it at
+           runtime changed nothing because the plugin reads it once at init.
+           It is not the reason the carriage used to sit still - see the
+           initial_value note below - so the gain is left at the default. -->
       <command_interface name="position">
         <param name="min">0.05</param>
         <param name="max">0.8</param>
-        <param name="position_proportional_gain">20.0</param>
       </command_interface>
+      <!-- Start just ABOVE the lower limit, never on it. Measured 15. 9.: the
+           carriage drives onto the 0.05 hard stop from above without trouble
+           (150 mm in one move), but once it rests exactly there the position
+           interface cannot move it again in EITHER direction - 0.00 mm against
+           a 0.20 m command, while the action still reports success. Ignition
+           realises a position command as a joint velocity, and at the limit
+           that velocity is zeroed. Spawning at 0.05 therefore started the robot
+           already locked, which is what P-13 has been chasing since 30. 6. -->
       <state_interface name="position">
-        <param name="initial_value">0.05</param>
+        <param name="initial_value">0.06</param>
       </state_interface>
       <state_interface name="velocity"/>
@@ -362,8 +415,15 @@
         <param name="min">0.05</param>
         <param name="max">0.8</param>
-        <param name="position_proportional_gain">20.0</param>
       </command_interface>
+      <!-- Start just ABOVE the lower limit, never on it. Measured 15. 9.: the
+           carriage drives onto the 0.05 hard stop from above without trouble
+           (150 mm in one move), but once it rests exactly there the position
+           interface cannot move it again in EITHER direction - 0.00 mm against
+           a 0.20 m command, while the action still reports success. Ignition
+           realises a position command as a joint velocity, and at the limit
+           that velocity is zeroed. Spawning at 0.05 therefore started the robot
+           already locked, which is what P-13 has been chasing since 30. 6. -->
       <state_interface name="position">
-        <param name="initial_value">0.05</param>
+        <param name="initial_value">0.06</param>
       </state_interface>
       <state_interface name="velocity"/>
