Commit message: fix: resolve URDF material conflicts, wheel mesh compatibility and controller spawner timeouts

File: src/pas_dual_arm_bringup/urdf/base/wheel.urdf.xacro (robot description, xacro)
@@ -60,5 +60,5 @@
           </xacro:if>
           <xacro:unless value="${sagital_reflect == 1}">
-            <mesh filename="package://omni_base_description/meshes/wheels/wheel_link_reverted.stl" scale="1 1 1"/>
+            <mesh filename="package://omni_base_description/meshes/wheels/wheel_link_reflected.stl" scale="1 1 1"/>
           </xacro:unless>
         </geometry>

File: src/pas_dual_arm_bringup/urdf/robot.urdf.xacro (robot description, xacro)
@@ -16,4 +16,6 @@
   <xacro:property name="namespace" value=""/>
   <xacro:property name="is_public_sim" value="true"/>
+  <!-- Prevent duplicate aluminum/plastic material definitions between pal_urdf_utils (>=2.11) and realsense2_description -->
+  <xacro:property name="realsense_materials_defined" value="true" scope="global"/>
   <!-- pal_urdf_utils laser/sensor macros branch on this; we skip omni_base.urdf.xacro
        (see note above) so it's never set upstream. Anything != 'classic' is correct
